File: AiO_Micro45_XIAO_C3/AiO_Micro45_XIAO_C3.kicad_pcb (KiCad board)
At the start: 2 copper layers, 27.3 x 24.4 mm, 7 parts, among them J1 PZ200-1-10-Z (1x10 male 2.00 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, J2 PZ200-1-10-Z (1x10 male 2.00 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, J3 PM254-1-07-Z-8.5 (1x07 female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, J4 PM254-1-07-Z-8.5 (1x07 female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

Commit message: Micro XIAO adapter v1.2: ideal diode on the XIAO 3.3 V, 1k serial resistors
- U2 (TI LM66100, SC-70-6, CE tied to VOUT) between the AiO 3.3 V and the
  XIAO 3V3 pin, plus C2 22 uF on the XIAO side. The XIAO USB-C can now be
  plugged in with the adapter on the Micro without feeding the AiO 3.3 V.
- R1, R2 100R -> 1k (C17513), as on the Standard adapter, to limit the
  current into an unpowered Teensy RX2.
- Same outline, header holes and XIAO position; 2 new vias.
- Regenerated Gerber zip, BOM/CPL (both sides and top only), schematic PDF
  and board picture. KiCad 7 DRC: 0 errors; schematic netlist = PCB.

Co-Authored-By: Claude Opus 5.5 (1M context) <noreply@anthropic.com>
Claude-Session: https://claude.ai/code/session_01YVKLpV6sqQR2BVk9gW2JwB
Parts:
- added C2: 22uF, AiO_XIAO_Adapter:C_0805_2012Metric, F.Cu at (102.0, 103.7)
- added U2: LM66100DCKR, AiO_XIAO_Adapter:SOT-363_SC-70-6, F.Cu at (105.0, 104.0)
- R1, R2: value 100 -> 1k
Connections:
- J4 pad 5: +3V3 -> /XIAO_3V3
Routing:
- net +3V3: track 17.4 -> 30.5 mm, vias 0 -> 1
- net /XIAO_3V3: track 0.00 -> 11.1 mm
- net GND: track 1.20 -> 2.45 mm, vias 8 -> 9
Other:
- board text added: "C2"
- board text added: "U2"
- board text added: "v1.2 2026-10"
- board text removed: "v1.1 2026-10"
