File: AiO_Micro45_XIAO_C3/AiO_Micro45_XIAO_C3.kicad_sch (KiCad schematic)
At the start: 7 parts, among them J1 PZ200-1-10-Z (1x10 male 2.00 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, J2 PZ200-1-10-Z (1x10 male 2.00 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, J3 PM254-1-07-Z-8.5 (1x07 female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, J4 PM254-1-07-Z-8.5 (1x07 female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

Commit message: Micro XIAO adapter v1.2: ideal diode on the XIAO 3.3 V, 1k serial resistors
- U2 (TI LM66100, SC-70-6, CE tied to VOUT) between the AiO 3.3 V and the
  XIAO 3V3 pin, plus C2 22 uF on the XIAO side. The XIAO USB-C can now be
  plugged in with the adapter on the Micro without feeding the AiO 3.3 V.
- R1, R2 100R -> 1k (C17513), as on the Standard adapter, to limit the
  current into an unpowered Teensy RX2.
- Same outline, header holes and XIAO position; 2 new vias.
- Regenerated Gerber zip, BOM/CPL (both sides and top only), schematic PDF
  and board picture. KiCad 7 DRC: 0 errors; schematic netlist = PCB.

Co-Authored-By: Claude Opus 5.5 (1M context) <noreply@anthropic.com>
Claude-Session: https://claude.ai/code/session_01YVKLpV6sqQR2BVk9gW2JwB
Parts:
- added C2: 22uF, AiO_XIAO_Adapter:C_0805_2012Metric, symbol Device:C
- added U2: LM66100DCKR, AiO_XIAO_Adapter:SOT-363_SC-70-6, symbol AiO_XIAO_Adapter:LM66100
- R1, R2: value 100 -> 1k; LCSC C17408 -> C17513
Connections:
- net +3V3: now also U2.1 (VIN); no longer J4.5 (3V3)
- net GND: now also C2.2, U2.2 (GND)
- new net XIAO_3V3: C2.1, J4.5 (3V3), U2.3 (~{CE}), U2.6 (VOUT)
- no-connect marks 25 -> 27
Other:
- note added: "Power: the 3.3 V of the socket (the board's 1 A K7803M regulator) goes through U2 (LM66100 ideal diode) into the XIAO 3V3 pin. U2 stops the XIAO USB from feeding the AiO 3.3 V."
- note added: "R1 and R2: 1k in series on the serial lines (they limit the current into an unpowered Teensy to about 3 mA). On the ESP32-C3: Serial0 = D6 TX (GPIO21) and D7 RX (GPIO20)."
- note removed: "Power: the 3.3 V of the socket (the board's 1 A K7803M regulator) goes into the XIAO 3V3 pin. Do not plug in the XIAO USB-C with the adapter on the board."
- note removed: "R1 and R2: 100 ohm in series on the serial lines (protection). On the ESP32-C3: Serial0 = D6 TX (GPIO21) and D7 RX (GPIO20)."
Changed lines of the file:
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@@
   (title_block
     (title "AiO v4.5 Micro - XIAO ESP32C3 adapter (GPS2 / Serial2)")
-    (date "2026-10-19")
-    (rev "1.1")
+    (date "2026-10-20")
+    (rev "1.2")
     (company "renatorgr")
     (comment 1 "GPS2 socket pins copied from the official AiO v4.5 Micro PCB")
@@
   (no_connect (at 223.52 121.92))
   (wire (pts (xy 223.52 124.46) (xy 228.60 124.46)) (stroke (width 0) (type default)))
-  (symbol (lib_id "power:+3V3") (at 228.60 124.46 0) (unit 1)
-    (in_bom yes) (on_board yes) (dnp no)
-    (property "Reference" "#PWR04" (at 228.60 129.46 0) (effects (font (size 1.27 1.27)) hide))
-    (property "Value" "+3V3" (at 228.60 120.65 0) (effects (font (size 1.27 1.27))))
-    (property "Footprint" "" (at 228.60 124.46 0) (effects (font (size 1.27 1.27)) hide))
-    (property "Datasheet" "" (at 228.60 124.46 0) (effects (font (size 1.27 1.27)) hide))
-    (pin "1")
-    (instances (project "AiO_Micro45_XIAO_C3" (path "/4f6b7c2e-9a51-4d1e-8c1a-5a3c0e7d2b10" (reference "#PWR04") (unit 1))))
-  )
+  (label "XIAO_3V3" (at 228.60 124.46 0) (fields_autoplaced) (effects (font (size 1.27 1.27)) (justify left bottom)))
   (wire (pts (xy 223.52 127.00) (xy 228.60 127.00)) (stroke (width 0) (type default)))
   (wire (pts (xy 228.60 127.00) (xy 231.14 127.00)) (stroke (width 0) (type default)))
@@
     (in_bom yes) (on_board yes) (dnp no)
     (property "Reference" "R1" (at 130.81 74.93 0) (effects (font (size 1.27 1.27)) (justify left)))
-    (property "Value" "100" (at 130.81 77.47 0) (effects (font (size 1.27 1.27)) (justify left)))
+    (property "Value" "1k" (at 130.81 77.47 0) (effects (font (size 1.27 1.27)) (justify left)))
     (property "Footprint" "AiO_XIAO_Adapter:R_0805_2012Metric" (at 127.0 76.2 0) (effects (font (size 1.27 1.27)) hide))
     (property "Datasheet" "~" (at 127.0 76.2 0) (effects (font (size 1.27 1.27)) hide))
-    (property "LCSC" "C17408" (at 127.0 76.2 0) (effects (font (size 1.27 1.27)) hide))
+    (property "LCSC" "C17513" (at 127.0 76.2 0) (effects (font (size 1.27 1.27)) hide))
     (pin "1")
     (pin "2")
@@
     (in_bom yes) (on_board yes) (dnp no)
     (property "Reference" "R2" (at 153.67000000000002 74.93 0) (effects (font (size 1.27 1.27)) (justify left)))
-    (property "Value" "100" (at 153.67000000000002 77.47 0) (effects (font (size 1.27 1.27)) (justify left)))
+    (property "Value" "1k" (at 153.67000000000002 77.47 0) (effects (font (size 1.27 1.27)) (justify left)))
     (property "Footprint" "AiO_XIAO_Adapter:R_0805_2012Metric" (at 149.86 76.2 0) (effects (font (size 1.27 1.27)) hide))
     (property "Datasheet" "~" (at 149.86 76.2 0) (effects (font (size 1.27 1.27)) hide))
-    (property "LCSC" "C17408" (at 149.86 76.2 0) (effects (font (size 1.27 1.27)) hide))
+    (property "LCSC" "C17513" (at 149.86 76.2 0) (effects (font (size 1.27 1.27)) hide))
     (pin "1")
     (pin "2")
@@
     (instances (project "AiO_Micro45_XIAO_C3" (path "/4f6b7c2e-9a51-4d1e-8c1a-5a3c0e7d2b10" (reference "#PWR07") (unit 1))))
   )
+  (symbol (lib_id "AiO_XIAO_Adapter:LM66100") (at 101.6 116.84 0) (unit 1)
+    (in_bom yes) (on_board yes) (dnp no)
+    (property "Reference" "U2" (at 101.6 109.22 0) (effects (font (size 1.27 1.27))))
+    (property "Value" "LM66100DCKR" (at 101.6 106.68 0) (effects (font (size 1.27 1.27))))
+    (property "Footprint" "AiO_XIAO_Adapter:SOT-363_SC-70-6" (at 101.6 116.84 0) (effects (font (size 1.27 1.27)) hide))
+    (property "Datasheet" "https://www.ti.com/lit/ds/symlink/lm66100.pdf" (at 101.6 116.84 0) (effects (font (size 1.27 1.27)) hide))
+    (property "LCSC" "C2869734" (at 101.6 116.84 0) (effects (font (size 1.27 1.27)) hide))
+    (property "Note" "Ideal diode: the AiO 3.3 V feeds the XIAO, the XIAO USB cannot feed the AiO. CE tied to VOUT" (at 101.6 116.84 0) (effects (font (size 1.27 1.27)) hide))
+    (pin "1")
+    (pin "2")
+    (pin "3")
+    (pin "4")
+    (pin "5")
+    (pin "6")
+    (instances (project "AiO_Micro45_XIAO_C3" (path "/4f6b7c2e-9a51-4d1e-8c1a-5a3c0e7d2b10" (reference "U2") (unit 1))))
+  )
+  (wire (pts (xy 91.44 114.30) (xy 88.90 114.30)) (stroke (width 0) (type default)))
+  (symbol (lib_id "power:+3V3") (at 88.90 114.30 0) (unit 1)
+    (in_bom yes) (on_board yes) (dnp no)
+    (property "Reference" "#PWR08" (at 88.90 119.30 0) (effects (font (size 1.27 1.27)) hide))
+    (property "Value" "+3V3" (at 88.90 110.49 0) (effects (font (size 1.27 1.27))))
+    (property "Footprint" "" (at 88.90 114.30 0) (effects (font (size 1.27 1.27)) hide))
+    (property "Datasheet" "" (at 88.90 114.30 0) (effects (font (size 1.27 1.27)) hide))
+    (pin "1")
+    (instances (project "AiO_Micro45_XIAO_C3" (path "/4f6b7c2e-9a51-4d1e-8c1a-5a3c0e7d2b10" (reference "#PWR08") (unit 1))))
+  )
+  (wire (pts (xy 111.76 114.30) (xy 114.30 114.30)) (stroke (width 0) (type default)))
+  (label "XIAO_3V3" (at 114.30 114.30 0) (fields_autoplaced) (effects (font (size 1.27 1.27)) (justify left bottom)))
+  (wire (pts (xy 111.76 116.84) (xy 114.30 116.84)) (stroke (width 0) (type default)))
+  (label "XIAO_3V3" (at 114.30 116.84 0) (fields_autoplaced) (effects (font (size 1.27 1.27)) (justify left bottom)))
+  (no_connect (at 111.76 119.38))
+  (no_connect (at 91.44 119.38))
+  (wire (pts (xy 101.60 124.46) (xy 101.60 127.00)) (stroke (width 0) (type default)))
+  (symbol (lib_id "power:GND") (at 101.60 127.00 0) (unit 1)
+    (in_bom yes) (on_board yes) (dnp no)
+    (property "Reference" "#PWR09" (at 101.60 132.00 0) (effects (font (size 1.27 1.27)) hide))
+    (property "Value" "GND" (at 101.60 130.81 0) (effects (font (size 1.27 1.27))))
+    (property "Footprint" "" (at 101.60 127.00 0) (effects (font (size 1.27 1.27)) hide))
+    (property "Datasheet" "" (at 101.60 127.00 0) (effects (font (size 1.27 1.27)) hide))
+    (pin "1")
+    (instances (project "AiO_Micro45_XIAO_C3" (path "/4f6b7c2e-9a51-4d1e-8c1a-5a3c0e7d2b10" (reference "#PWR09") (unit 1))))
+  )
+  (symbol (lib_id "Device:C") (at 165.1 116.84 0) (unit 1)
+    (in_bom yes) (on_board yes) (dnp no)
+    (property "Reference" "C2" (at 168.91 115.57 0) (effects (font (size 1.27 1.27)) (justify left)))
+    (property "Value" "22uF" (at 168.91 118.11 0) (effects (font (size 1.27 1.27)) (justify left)))
+    (property "Footprint" "AiO_XIAO_Adapter:C_0805_2012Metric" (at 165.1 116.84 0) (effects (font (size 1.27 1.27)) hide))
+    (property "Datasheet" "~" (at 165.1 116.84 0) (effects (font (size 1.27 1.27)) hide))
+    (property "LCSC" "C45783" (at 165.1 116.84 0) (effects (font (size 1.27 1.27)) hide))
+    (pin "1")
+    (pin "2")
+    (instances (project "AiO_Micro45_XIAO_C3" (path "/4f6b7c2e-9a51-4d1e-8c1a-5a3c0e7d2b10" (reference "C2") (unit 1))))
+  )
+  (wire (pts (xy 165.10 113.03) (xy 165.10 110.49)) (stroke (width 0) (type default)))
+  (label "XIAO_3V3" (at 165.10 110.49 0) (fields_autoplaced) (effects (font (size 1.27 1.27)) (justify left bottom)))
+  (wire (pts (xy 165.10 120.65) (xy 165.10 123.19)) (stroke (width 0) (type default)))
+  (symbol (lib_id "power:GND") (at 165.10 123.19 0) (unit 1)
+    (in_bom yes) (on_board yes) (dnp no)
+    (property "Reference" "#PWR10" (at 165.10 128.19 0) (effects (font (size 1.27 1.27)) hide))
+    (property "Value" "GND" (at 165.10 127.00 0) (effects (font (size 1.27 1.27))))
+    (property "Footprint" "" (at 165.10 123.19 0) (effects (font (size 1.27 1.27)) hide))
+    (property "Datasheet" "" (at 165.10 123.19 0) (effects (font (size 1.27 1.27)) hide))
+    (pin "1")
+    (instances (project "AiO_Micro45_XIAO_C3" (path "/4f6b7c2e-9a51-4d1e-8c1a-5a3c0e7d2b10" (reference "#PWR10") (unit 1))))
+  )
   (text "XIAO ESP32C3 adapter for the GPS2 socket (Dual-Left, U11) of the AiO v4.5 Micro" (at 25.40 25.40 0) (effects (font (size 2.0 2.0)) (justify left bottom)))
   (text "GPS2 socket: pin 2 = Teensy RX2 (pin 7), pin 3 = Teensy TX2 (pin 8). On the Teensy it is Serial2." (at 25.40 31.75 0) (effects (font (size 1.27 1.27)) (justify left bottom)))
-  (text "Power: the 3.3 V of the socket (the board's 1 A K7803M regulator) goes into the XIAO 3V3 pin. Do not plug in the XIAO USB-C with the adapter on the board." (at 25.40 35.56 0) (effects (font (size 1.27 1.27)) (justify left bottom)))
-  (text "R1 and R2: 100 ohm in series on the serial lines (protection). On the ESP32-C3: Serial0 = D6 TX (GPIO21) and D7 RX (GPIO20)." (at 25.40 39.37 0) (effects (font (size 1.27 1.27)) (justify left bottom)))
+  (text "Power: the 3.3 V of the socket (the board's 1 A K7803M regulator) goes through U2 (LM66100 ideal diode) into the XIAO 3V3 pin. U2 stops the XIAO USB from feeding the AiO 3.3 V." (at 25.40 35.56 0) (effects (font (size 1.27 1.27)) (justify left bottom)))
+  (text "R1 and R2: 1k in series on the serial lines (they limit the current into an unpowered Teensy to about 3 mA). On the ESP32-C3: Serial0 = D6 TX (GPIO21) and D7 RX (GPIO20)." (at 25.40 39.37 0) (effects (font (size 1.27 1.27)) (justify left bottom)))
   (text "Not connected: pins 6 to 8 (F9P USB), 16 (wired to the GPS1 socket), 18 (LED RTK_STAT_1) and the other NC pins." (at 25.40 43.18 0) (effects (font (size 1.27 1.27)) (justify left bottom)))
   (text "J1 = socket pins 1-10, J2 = socket pins 11-20 (J2 pin 1 = socket pin 11). Both are 1x10 2.00 mm male headers on the bottom side." (at 25.40 46.99 0) (effects (font (size 1.27 1.27)) (justify left bottom)))
