File: Relay24_ESP32/Relay24_ESP32.kicad_sch (KiCad schematic)
At the start: 67 parts, among them J25 12V IN, J26 12V ACT A (left), J27 12V ACT A (right), J28 12V ACT B (left), J29 12V ACT B (right), J30 DevKitC J2 (3V3..5V), J31 DevKitC J3 (GND..CLK), J32 HR911105A, J33 I2C, J34 Analog, U1 74HC595, U2 74HC595, U3 74HC595, U4 ULN2803A, U5 ULN2803A, U6 ULN2803A, U7 LM2596S-5.0, U8 AMS1117-3.3, U9 LAN8720A

Commit message: Relay24_ESP32: fix wrong LCSC numbers and fill the missing ones
The JLCPCB BOM check showed parts with no LCSC number (sockets, headers,
RBIAS resistor) and parts in shortfall. Two numbers were wrong parts:
C6116 is a 74LVT244 in SSOP-20, not a ULN2803A, and C23182 is 47 ohm, not
49.9 ohm; C22374 no longer exists.

- U4-U6: Shanghai Belling ULN2803 SOP-18 300 mil (C22437476)
- D1-D24, D31: XINGLIGHT XL-1608SYGC-06 (C965805); D30: XL-1608UYC-06 (C965802)
- R31: Yageo RC0603FR-0712K1L 12.1k 1% (C123417); R38-R41: 49.9 ohm (C23185)
- J30/J31: 1x19 female header (C319202); J33/J34: 1x4 pin header (C124378)
- D26 SMBJ18A (C151256), C25 100uF 50V (C97812), C26 220uF 25V (C165536),
  L1 CYH127-33UH (C2929502)

Only the part fields changed on the routed board (DRC still 0 errors,
0 unconnected); BOM/CPL, schematic and views regenerated. README notes
the second sources and the L1 land pattern to check.

Co-Authored-By: Claude Opus 5.5 <noreply@anthropic.com>
Claude-Session: https://claude.ai/code/session_01VKEBDGHaGvWUQ7R6BJeKCx
Parts:
- C25: LCSC (none) -> C97812
- C26: LCSC (none) -> C165536
- D26: LCSC (none) -> C151256
- D30: LCSC C72038 -> C965802
- D31: LCSC C72043 -> C965805
- J30, J31: LCSC (none) -> C319202
- J33, J34: LCSC (none) -> C124378
- L1: LCSC (none) -> C2929502
- R31: LCSC C22374 -> C123417
- R38, R39, R40, R41: LCSC C23182 -> C23185
- U4, U5, U6: LCSC C6116 -> C22437476

Commit message: Relay24_ESP32: replace the LAN8720A with an RTL8201F (Economic PCBA)
JLCPCB assembles the LAN8720A (C45223) only on its Standard service,
so the Ethernet PHY is now a Realtek RTL8201F-VB-CG (C45044, QFN-32),
which is on the Economic service.

- RTL8201F runs on a 25 MHz crystal (Y1, C9006, 2x 18 pF C1647) and
  sends the 50 MHz RMII reference clock out of TXC through R30 (33 ohm)
  to GPIO0 (ETH_CLOCK_GPIO0_IN); GPIO17 is free again.
- Straps: RXDV pulled up (RMII), LED0/LED1 pulled down (PHY address 0,
  active-high LEDs). D30 shows a 10 Mbit link, D31 a 100 Mbit link.
- RSET 2.49k (C136931), PHYRSTB held low by R33 until GPIO33 is set.
- MDI pair 0 to RJ45 pins 1-2 and pair 1 to pins 3-6 (standard wiring),
  49.9 ohm terminations to 3V3 kept; new fan-out and pre-route for the
  QFN in make_pcb.py; custom schematic symbol in make_sch.py.
- router.py: the flood fill that finds existing copper of a net is now
  8-connected, so a diagonal fixed track is one piece of copper and the
  router no longer adds a wide stub next to it (clearance violation).
- make_pcb.py: RELAY24_FIXED_ONLY=1 builds only the hand-placed copper
  and runs the DRC, for quick checks.
- README, schematic, board, Gerber, BOM, CPL and views regenerated.
  Router failures 0, DRC 0 errors / 0 unconnected. Nothing built yet.

Co-Authored-By: Claude Fable 5.1 <noreply@anthropic.com>
Claude-Session: https://claude.ai/code/session_01VKEBDGHaGvWUQ7R6BJeKCx
Parts:
- removed R37: 10k, Resistor_SMD:R_0603_1608Metric, symbol Device:R
- removed U9: LAN8720A, Package_DFN_QFN:VQFN-24-1EP_4x4mm_P0.5mm_EP2.5x2.5mm_ThermalVias, symbol Interface_Ethernet:LAN8720A
- added C38: 10uF, Capacitor_SMD:C_0805_2012Metric, symbol Device:C
- added U9: RTL8201F, Package_DFN_QFN:QFN-32-1EP_5x5mm_P0.5mm_EP3.45x3.45mm_ThermalVias, symbol Relay24:RTL8201F
- added Y1: 25MHz, Crystal:Crystal_SMD_3225-4Pin_3.2x2.5mm, symbol Device:Crystal_GND24
- C34: value 1uF -> 18pF; LCSC C15849 -> C1647
- C35: value 10uF -> 18pF; footprint Capacitor_SMD:C_0805_2012Metric -> Capacitor_SMD:C_0603_1608Metric; LCSC C15850 -> C1647
- R31: value 12.1k 1% -> 2.49k 1%; LCSC C123417 -> C136931
- R32, R35, R36: value 10k -> 4.7k; LCSC C25804 -> C23162
Connections:
- net ETH_CLKIN is gone; now on net ETH_CLK: R30.2
- net PHYAD0 is gone; now on net GND: R32.1
- net +3V3: now also C38.1, U9.14 (DVDD33), U9.30 (AVDD33), U9.7 (AVDD33); no longer C32.1, C35.1, J30.10 (Pin_10), J30.11 (Pin_11), J32.1, J32.3, J32.6, R36.1, R36.2, R39.1, R40.1, R41.1, R43.1
- net ETH_CLK: now also J31.14 (Pin_14); no longer J31.11 (Pin_11), R30.1
- net ETH_RST: now also U9.21 (PHYRSTB)
- net GND: now also R36.1, R43.2, C38.2, U9.33 (EP/GND), Y1.2, Y1.4; no longer R32.2
- net RMII_MDC: now also U9.22 (MDC)
- net RMII_MDIO: now also U9.23 (MDIO)
- net RMII_RXD0: now also U9.9 (RXD0); no longer R35.1
- net RMII_TXD0: now also U9.16 (TXD0)
- net RMII_TXD1: now also U9.17 (TXD1)
- net RMII_TXEN: now also U9.20 (TXEN)
- net LED_LNK renamed PHY_LED0
- net PHY_LED0: now also R32.2, U9.24 (LED0/PHYAD0)
- net LED_LNK_K renamed LED0_K
- net LED_SPD renamed LED1_K
- net LED1_K: now also R43.1
- net LED_SPD_A renamed PHY_LED1
- net PHY_LED1: now also R36.2, U9.25 (LED1/PHYAD1); no longer R43.2
- net RBIAS renamed RSET
- net RSET: now also U9.1 (RSET)
- net TXP renamed MDI0N
- net MDI0N: now also U9.4 (MDI-[0])
- net VDDCR renamed DVDD10
- net DVDD10: now also U9.29 (DVDD10OUT); no longer C34.1
- new net AVDD10: C32.1, U9.2 (AVDD10OUT)
- new net ETH_REFCLK: R30.1, U9.15 (TXC/REF_CLK)
- new net MDI0P: J32.1, R39.1, U9.3 (MDI+[0])
- new net MDI1N: J32.6, R40.1, U9.6 (MDI-[1])
- new net MDI1P: J32.3, R41.1, U9.5 (MDI+[1])
- new net PHY_RXDV: R35.1, U9.8 (RXDV)
- new net RMII_CRS_DV: J30.11 (Pin_11), U9.26 (CRS_DV)
- new net RMII_RXD1: J30.10 (Pin_10), U9.10 (RXD1)
- new net XTAL1: C34.1, U9.31 (CKXTAL1), Y1.1
- new net XTAL2: C35.1, U9.32 (CKXTAL2), Y1.3
- no-connect marks 23 -> 28
Other:
- note added: "ESP32 DevKitC V4 (38 pins) in two 1x19 sockets. RMII pins are fixed by the ESP32: TXD0 19, TXD1 22, TXEN 21, RXD0 25, RXD1 26, CRS_DV 27, MDC 23, MDIO 18, 50 MHz reference clock in on GPIO0 (from the PHY)."
- note added: "RJ45 HR911105A: PHY pair 0 (transmit) on pins 1-2, pair 1 (receive) on 3-6, centre taps (4, 5, 7, 8) to 3.3 V with C36/C37, its own LEDs unused."
- note added: "RTL8201F on a 25 MHz crystal (Y1, C34/C35); the 50 MHz RMII clock comes OUT of TXC -> R30 -> GPIO0 (ETH_CLOCK_GPIO0_IN). R33 keeps the PHY in reset until GPIO33 is high, so GPIO0 is free at boot."
- note added: "Straps: RXDV up (R35) = RMII; LED0/LED1 down (R32/R36) = PHY address 0, LEDs active high: D30 = 10 Mbit link/activity, D31 = 100 Mbit (default LED mode). RSET 2.49 k (R31). 49.9 ohm terminations to 3.3 V (R38-R41)."
- note removed: "ESP32 DevKitC V4 (38 pins) in two 1x19 sockets. RMII pins are fixed by the ESP32: TXD0 19, TXD1 22, TXEN 21, RXD0 25, RXD1 26, CRS_DV 27, MDC 23, MDIO 18, 50 MHz clock out on GPIO17."
- note removed: "LAN8720A in REF_CLK-in mode (no crystal): GPIO17 -> R30 -> CLKIN. PHY address 0 (R32). Straps: MODE 111 (R35-R37), REGOFF low (LED1 to GND), nINTSEL high (LED2 from 3.3 V)."
- note removed: "RJ45 HR911105A: pairs 1-2 and 3-6, centre taps (4, 5, 7, 8) to 3.3 V with C36/C37, its own LEDs unused (D30/D31 on the board)."

Commit message: Relay24_ESP32: use a 5032 two-pin crystal that JLCPCB assembles normally
JLCPCB flags the 3225 four-pin crystal (C9006) as "Assembly Difficulty:
High" and warned that it may cost extra. Y1 is now the YXC X503225MSB2GI
(C112569, 25 MHz, 5.0 x 3.2 mm, two pins, CL 20 pF), which carries no
such flag.

- Load capacitors C34/C35 go from 18 pF to 33 pF (C1663, basic part)
  to match the 20 pF load capacitance.
- The crystal sits below the PHY, XTAL1 straight down from pin 31,
  XTAL2 from pin 32, each load capacitor right under its pad; the
  ground stubs and vias of the old crystal are gone.
- Schematic, board, Gerber, BOM, CPL, views and README regenerated.
  Router failures 0, DRC 0 errors / 0 unconnected.

Co-Authored-By: Claude Opus 5.5 <noreply@anthropic.com>
Claude-Session: https://claude.ai/code/session_01VKEBDGHaGvWUQ7R6BJeKCx
Parts:
- removed Y1: 25MHz, Crystal:Crystal_SMD_3225-4Pin_3.2x2.5mm, symbol Device:Crystal_GND24
- added Y1: 25MHz, Crystal:Crystal_SMD_5032-2Pin_5.0x3.2mm, symbol Device:Crystal
- C34, C35: value 18pF -> 33pF; LCSC C1647 -> C1663
Connections:
- net XTAL1: now also Y1.1
- net XTAL2: now also Y1.2
