File: Relay24_ESP32/relays_17_24.kicad_sch (KiCad schematic)
At the start: 32 parts, among them J17 Section 17, J18 Section 18, J19 Section 19, J20 Section 20, J21 Section 21, J22 Section 22, J23 Section 23, J24 Section 24, K17 HF115F/012-2ZS4, K18 HF115F/012-2ZS4, K19 HF115F/012-2ZS4, K20 HF115F/012-2ZS4, K21 HF115F/012-2ZS4, K22 HF115F/012-2ZS4, K23 HF115F/012-2ZS4, K24 HF115F/012-2ZS4

Commit message: Relay24_ESP32: fix wrong LCSC numbers and fill the missing ones
The JLCPCB BOM check showed parts with no LCSC number (sockets, headers,
RBIAS resistor) and parts in shortfall. Two numbers were wrong parts:
C6116 is a 74LVT244 in SSOP-20, not a ULN2803A, and C23182 is 47 ohm, not
49.9 ohm; C22374 no longer exists.

- U4-U6: Shanghai Belling ULN2803 SOP-18 300 mil (C22437476)
- D1-D24, D31: XINGLIGHT XL-1608SYGC-06 (C965805); D30: XL-1608UYC-06 (C965802)
- R31: Yageo RC0603FR-0712K1L 12.1k 1% (C123417); R38-R41: 49.9 ohm (C23185)
- J30/J31: 1x19 female header (C319202); J33/J34: 1x4 pin header (C124378)
- D26 SMBJ18A (C151256), C25 100uF 50V (C97812), C26 220uF 25V (C165536),
  L1 CYH127-33UH (C2929502)

Only the part fields changed on the routed board (DRC still 0 errors,
0 unconnected); BOM/CPL, schematic and views regenerated. README notes
the second sources and the L1 land pattern to check.

Co-Authored-By: Claude Opus 5.5 <noreply@anthropic.com>
Claude-Session: https://claude.ai/code/session_01VKEBDGHaGvWUQ7R6BJeKCx
Parts:
- D17, D18, D19, D20, D21, D22, D23, D24: LCSC C72043 -> C965805
