File: Relay24_ESP32/relays_9_16.kicad_sch (KiCad schematic)
At the start: 32 parts, among them J10 Section 10, J11 Section 11, J12 Section 12, J13 Section 13, J14 Section 14, J15 Section 15, J16 Section 16, J9 Section 9, K10 HF115F/012-2ZS4, K11 HF115F/012-2ZS4, K12 HF115F/012-2ZS4, K13 HF115F/012-2ZS4, K14 HF115F/012-2ZS4, K15 HF115F/012-2ZS4, K16 HF115F/012-2ZS4, K9 HF115F/012-2ZS4

Commit message: Relay24_ESP32: fix wrong LCSC numbers and fill the missing ones
The JLCPCB BOM check showed parts with no LCSC number (sockets, headers,
RBIAS resistor) and parts in shortfall. Two numbers were wrong parts:
C6116 is a 74LVT244 in SSOP-20, not a ULN2803A, and C23182 is 47 ohm, not
49.9 ohm; C22374 no longer exists.

- U4-U6: Shanghai Belling ULN2803 SOP-18 300 mil (C22437476)
- D1-D24, D31: XINGLIGHT XL-1608SYGC-06 (C965805); D30: XL-1608UYC-06 (C965802)
- R31: Yageo RC0603FR-0712K1L 12.1k 1% (C123417); R38-R41: 49.9 ohm (C23185)
- J30/J31: 1x19 female header (C319202); J33/J34: 1x4 pin header (C124378)
- D26 SMBJ18A (C151256), C25 100uF 50V (C97812), C26 220uF 25V (C165536),
  L1 CYH127-33UH (C2929502)

Only the part fields changed on the routed board (DRC still 0 errors,
0 unconnected); BOM/CPL, schematic and views regenerated. README notes
the second sources and the L1 land pattern to check.

Co-Authored-By: Claude Opus 5.5 <noreply@anthropic.com>
Claude-Session: https://claude.ai/code/session_01VKEBDGHaGvWUQ7R6BJeKCx
Parts:
- D10, D11, D12, D13, D14, D15, D16, D9: LCSC C72043 -> C965805
